Commit message: added ros publisher

File: trial.urdf (robot description, URDF)
Before this commit: robot cart, 6 links, 5 joints
Links:
- removed link base_footprint
- removed link base_link
Joints:
- removed joint base_footprint_joint
- removed joint chassis_joint
- joint caster_wheel_joint: origin xyz=0.075 0 -0.013 -> xyz=0.28 0 -0.013
- joint left_wheel_joint: origin xyz=0 0.1485 0 rpy=-1.57 0 0 -> xyz=0.1 0.13 0 rpy=-1.57 0 0; parent base_link -> chassis
- joint right_wheel_joint: origin xyz=0 -0.1485 0 rpy=1.57 0 0 -> xyz=0.1 -0.13 0 rpy=1.57 0 0; parent base_link -> chassis
